Commit message: fix name is keyword

File: urdf_model_generator/urdf/test_robot.urdf (robot description, URDF)
Before this commit: robot r2d2, 17 links, 16 joints
Links:
- removed link box
- added link box_, mass 1; collision box size=.08 .08 .08; visual box size=.08 .08 .08
Joints:
- joint tobox: child box -> box_
